Commit message: Add visual CBF proxy volumes

File: ur_cbf_ws/src/ur_cbf_bringup/urdf/ur_rg2_gz.urdf.xacro (robot description, xacro)
@@ -19,4 +19,5 @@
   <xacro:arg name="simulation_controllers" default=""/>
   <xacro:arg name="ros_namespace" default=""/>
+  <xacro:arg name="show_cbf_volumes" default="$(optenv CBF_VOLUMES true)"/>
   <!-- O Xacro upstream declara gripper_tcp no escopo da inclusao. -->
   <xacro:property name="prefix" value="$(arg tf_prefix)"/>
@@ -24,4 +25,5 @@
   <xacro:include filename="$(find ur_simulation_gz)/urdf/ur_gz.ros2_control.xacro"/>
   <xacro:include filename="$(find onrobot_description)/urdf/rg2_macro.xacro"/>
+  <xacro:include filename="$(find ur_cbf_bringup)/urdf/cbf_visual_volumes.urdf.xacro"/>
   <link name="world"/>
   <link name="ground_plane">
@@ -57,4 +59,11 @@
     <origin xyz="0 0 0" rpy="0 0 ${-pi/2}"/>
   </joint>
+  <xacro:if value="$(arg show_cbf_volumes)">
+    <xacro:property name="selected_ur_type" value="$(arg ur_type)"/>
+    <xacro:if value="${selected_ur_type == 'ur3e'}">
+      <xacro:ur3e_cbf_visual_volumes prefix="$(arg tf_prefix)"/>
+    </xacro:if>
+    <xacro:rg2_cbf_visual_volume prefix="$(arg tf_prefix)"/>
+  </xacro:if>
   <gazebo reference="world"/>
   <gazebo>

File: ur_cbf_ws/src/ur_cbf_bringup/urdf/ur_rg6_gz.urdf.xacro (robot description, xacro)
@@ -19,4 +19,5 @@
   <xacro:arg name="simulation_controllers" default=""/>
   <xacro:arg name="ros_namespace" default=""/>
+  <xacro:arg name="show_cbf_volumes" default="$(optenv CBF_VOLUMES true)"/>
   <!-- O Xacro upstream declara gripper_tcp no escopo da inclusao. -->
   <xacro:property name="prefix" value="$(arg tf_prefix)"/>
@@ -24,4 +25,5 @@
   <xacro:include filename="$(find ur_simulation_gz)/urdf/ur_gz.ros2_control.xacro"/>
   <xacro:include filename="$(find onrobot_description)/urdf/rg6_macro.xacro"/>
+  <xacro:include filename="$(find ur_cbf_bringup)/urdf/cbf_visual_volumes.urdf.xacro"/>
   <link name="world"/>
   <link name="ground_plane">
@@ -57,4 +59,10 @@
     <origin xyz="0 0 0" rpy="0 0 ${-pi/2}"/>
   </joint>
+  <xacro:if value="$(arg show_cbf_volumes)">
+    <xacro:property name="selected_ur_type" value="$(arg ur_type)"/>
+    <xacro:if value="${selected_ur_type == 'ur3e'}">
+      <xacro:ur3e_cbf_visual_volumes prefix="$(arg tf_prefix)"/>
+    </xacro:if>
+  </xacro:if>
   <gazebo reference="world"/>
   <gazebo>
