Commit message: Correct UR3e proxy geometry and Gazebo visibility

File: ur_cbf_ws/src/ur_cbf_bringup/urdf/cbf_visual_volumes.urdf.xacro (robot description, xacro)
@@ -6,5 +6,6 @@
 -->
 <robot xmlns:xacro="http://wiki.ros.org/xacro">
-  <xacro:macro name="cbf_sphere_visual" params="name parent xyz radius rgba">
+  <xacro:macro name="cbf_sphere_visual"
+               params="name parent xyz radius rgba gazebo_visible">
     <link name="${name}_cbf_volume">
       <visual name="${name}_cbf_visual">
@@ -23,8 +24,16 @@
       <child link="${name}_cbf_volume"/>
     </joint>
+    <!-- RViz ignora a extensao gazebo; visibility_flags=0 oculta somente no SDF. -->
+    <xacro:unless value="${gazebo_visible}">
+      <gazebo reference="${name}_cbf_volume">
+        <visual>
+          <visibility_flags>0</visibility_flags>
+        </visual>
+      </gazebo>
+    </xacro:unless>
   </xacro:macro>
   <!-- Uma capsula e formada por um cilindro e duas esferas, todos visuais. -->
   <xacro:macro name="cbf_capsule_visual"
-               params="name parent center rpy cap_a cap_b radius length rgba">
+               params="name parent center rpy cap_a cap_b radius length rgba gazebo_visible">
     <link name="${name}_cbf_volume">
       <visual name="${name}_cbf_cylinder">
@@ -57,37 +66,73 @@
       <child link="${name}_cbf_volume"/>
     </joint>
+    <xacro:unless value="${gazebo_visible}">
+      <gazebo reference="${name}_cbf_volume">
+        <visual>
+          <visibility_flags>0</visibility_flags>
+        </visual>
+      </gazebo>
+    </xacro:unless>
   </xacro:macro>
-  <xacro:macro name="ur3e_cbf_visual_volumes" params="prefix">
+  <xacro:macro name="ur3e_cbf_visual_volumes" params="prefix gazebo_visible">
     <xacro:property name="arm_color" value="0.00 0.75 1.00 0.25"/>
+    <!--
+      Offsets fisicos da descricao oficial Jazzy do UR3e. Os eixos DH passam
+      pelas juntas, enquanto os corpos do braco e antebraco sao deslocados em z
+      nos respectivos frames de elo.
+    -->
+    <xacro:property name="shoulder_body_offset" value="0.120"/>
+    <xacro:property name="elbow_body_offset" value="0.027"/>
+    <xacro:property name="wrist_1_joint_offset" value="0.13105"/>
     <xacro:cbf_sphere_visual
       name="${prefix}base" parent="${prefix}base_link"
-      xyz="0 0 0.075" radius="0.110" rgba="${arm_color}"/>
+      xyz="0 0 0.075" radius="0.110" rgba="${arm_color}"
+      gazebo_visible="${gazebo_visible}"/>
     <xacro:cbf_sphere_visual
       name="${prefix}shoulder" parent="${prefix}shoulder_link"
-      xyz="0 0 0" radius="0.090" rgba="${arm_color}"/>
+      xyz="0 0 0" radius="0.090" rgba="${arm_color}"
+      gazebo_visible="${gazebo_visible}"/>
     <xacro:cbf_capsule_visual
       name="${prefix}upper_arm" parent="${prefix}upper_arm_link"
-      center="-0.121775 0 0" rpy="0 1.57079632679 0"
-      cap_a="0 0 0" cap_b="-0.24355 0 0"
-      radius="0.075" length="0.24355" rgba="${arm_color}"/>
+      center="-0.121775 0 ${shoulder_body_offset}" rpy="0 1.57079632679 0"
+      cap_a="0 0 ${shoulder_body_offset}"
+      cap_b="-0.24355 0 ${shoulder_body_offset}"
+      radius="0.075" length="0.24355" rgba="${arm_color}"
+      gazebo_visible="${gazebo_visible}"/>
     <xacro:cbf_sphere_visual
       name="${prefix}elbow" parent="${prefix}forearm_link"
-      xyz="0 0 0" radius="0.075" rgba="${arm_color}"/>
+      xyz="0 0 0" radius="0.075" rgba="${arm_color}"
+      gazebo_visible="${gazebo_visible}"/>
     <xacro:cbf_capsule_visual
       name="${prefix}forearm" parent="${prefix}forearm_link"
-      center="-0.1066 0 0" rpy="0 1.57079632679 0"
-      cap_a="0 0 0" cap_b="-0.2132 0 0"
-      radius="0.065" length="0.2132" rgba="${arm_color}"/>
+      center="-0.1066 0 ${elbow_body_offset}" rpy="0 1.57079632679 0"
+      cap_a="0 0 ${elbow_body_offset}"
+      cap_b="-0.2132 0 ${elbow_body_offset}"
+      radius="0.065" length="0.2132" rgba="${arm_color}"
+      gazebo_visible="${gazebo_visible}"/>
+    <!--
+      Completa o offset distal do antebraco ate o frame posterior a junta 4.
+      Comprimento: 0.13105 - 0.027 = 0.10405 m.
+    -->
+    <xacro:cbf_capsule_visual
+      name="${prefix}wrist_1_connector" parent="${prefix}forearm_link"
+      center="-0.2132 0 0.079025" rpy="0 0 0"
+      cap_a="-0.2132 0 ${elbow_body_offset}"
+      cap_b="-0.2132 0 ${wrist_1_joint_offset}"
+      radius="0.060" length="0.10405" rgba="${arm_color}"
+      gazebo_visible="${gazebo_visible}"/>
     <xacro:cbf_sphere_visual
       name="${prefix}wrist_1" parent="${prefix}wrist_1_link"
-      xyz="0 0 0" radius="0.060" rgba="${arm_color}"/>
+      xyz="0 0 0" radius="0.060" rgba="${arm_color}"
+      gazebo_visible="${gazebo_visible}"/>
     <xacro:cbf_sphere_visual
       name="${prefix}wrist_2" parent="${prefix}wrist_2_link"
-      xyz="0 0 0" radius="0.058" rgba="${arm_color}"/>
+      xyz="0 0 0" radius="0.058" rgba="${arm_color}"
+      gazebo_visible="${gazebo_visible}"/>
     <xacro:cbf_sphere_visual
       name="${prefix}wrist_3" parent="${prefix}wrist_3_link"
-      xyz="0 0 0" radius="0.058" rgba="${arm_color}"/>
+      xyz="0 0 0" radius="0.058" rgba="${arm_color}"
+      gazebo_visible="${gazebo_visible}"/>
   </xacro:macro>
-  <xacro:macro name="rg2_cbf_visual_volume" params="prefix">
+  <xacro:macro name="rg2_cbf_visual_volume" params="prefix gazebo_visible">
     <!-- Uma unica capsula cobre corpo, dedos e o TCP nominal da RG2. -->
     <xacro:cbf_capsule_visual
@@ -95,5 +140,6 @@
       center="0 0 0.110" rpy="0 0 0"
       cap_a="0 0 0.055" cap_b="0 0 0.165"
-      radius="0.090" length="0.110" rgba="1.00 0.45 0.00 0.30"/>
+      radius="0.090" length="0.110" rgba="1.00 0.45 0.00 0.30"
+      gazebo_visible="${gazebo_visible}"/>
   </xacro:macro>
 </robot>

File: ur_cbf_ws/src/ur_cbf_bringup/urdf/ur_rg2_gz.urdf.xacro (robot description, xacro)
@@ -20,4 +20,5 @@
   <xacro:arg name="ros_namespace" default=""/>
   <xacro:arg name="show_cbf_volumes" default="$(optenv CBF_VOLUMES true)"/>
+  <xacro:arg name="show_cbf_volumes_gazebo" default="$(optenv CBF_VOLUMES_GAZEBO true)"/>
   <!-- O Xacro upstream declara gripper_tcp no escopo da inclusao. -->
   <xacro:property name="prefix" value="$(arg tf_prefix)"/>
@@ -62,7 +63,11 @@
     <xacro:property name="selected_ur_type" value="$(arg ur_type)"/>
     <xacro:if value="${selected_ur_type == 'ur3e'}">
-      <xacro:ur3e_cbf_visual_volumes prefix="$(arg tf_prefix)"/>
+      <xacro:ur3e_cbf_visual_volumes
+        prefix="$(arg tf_prefix)"
+        gazebo_visible="$(arg show_cbf_volumes_gazebo)"/>
     </xacro:if>
-    <xacro:rg2_cbf_visual_volume prefix="$(arg tf_prefix)"/>
+    <xacro:rg2_cbf_visual_volume
+      prefix="$(arg tf_prefix)"
+      gazebo_visible="$(arg show_cbf_volumes_gazebo)"/>
   </xacro:if>
   <gazebo reference="world"/>

File: ur_cbf_ws/src/ur_cbf_bringup/urdf/ur_rg6_gz.urdf.xacro (robot description, xacro)
@@ -20,4 +20,5 @@
   <xacro:arg name="ros_namespace" default=""/>
   <xacro:arg name="show_cbf_volumes" default="$(optenv CBF_VOLUMES true)"/>
+  <xacro:arg name="show_cbf_volumes_gazebo" default="$(optenv CBF_VOLUMES_GAZEBO true)"/>
   <!-- O Xacro upstream declara gripper_tcp no escopo da inclusao. -->
   <xacro:property name="prefix" value="$(arg tf_prefix)"/>
@@ -62,5 +63,7 @@
     <xacro:property name="selected_ur_type" value="$(arg ur_type)"/>
     <xacro:if value="${selected_ur_type == 'ur3e'}">
-      <xacro:ur3e_cbf_visual_volumes prefix="$(arg tf_prefix)"/>
+      <xacro:ur3e_cbf_visual_volumes
+        prefix="$(arg tf_prefix)"
+        gazebo_visible="$(arg show_cbf_volumes_gazebo)"/>
     </xacro:if>
   </xacro:if>

Commit message: Remove redundant CBF proxy spheres

File: ur_cbf_ws/src/ur_cbf_bringup/urdf/cbf_visual_volumes.urdf.xacro (robot description, xacro)
@@ -25,4 +25,31 @@
     </joint>
     <!-- RViz ignora a extensao gazebo; visibility_flags=0 oculta somente no SDF. -->
+    <xacro:unless value="${gazebo_visible}">
+      <gazebo reference="${name}_cbf_volume">
+        <visual>
+          <visibility_flags>0</visibility_flags>
+        </visual>
+      </gazebo>
+    </xacro:unless>
+  </xacro:macro>
+  <!-- Cilindro sem tampas esfericas para ligar volumes ja sobrepostos. -->
+  <xacro:macro name="cbf_cylinder_visual"
+               params="name parent center rpy radius length rgba gazebo_visible">
+    <link name="${name}_cbf_volume">
+      <visual name="${name}_cbf_cylinder">
+        <origin xyz="${center}" rpy="${rpy}"/>
+        <geometry>
+          <cylinder radius="${radius}" length="${length}"/>
+        </geometry>
+        <material name="${name}_cbf_material">
+          <color rgba="${rgba}"/>
+        </material>
+      </visual>
+    </link>
+    <joint name="${name}_cbf_volume_joint" type="fixed">
+      <origin xyz="0 0 0" rpy="0 0 0"/>
+      <parent link="${parent}"/>
+      <child link="${name}_cbf_volume"/>
+    </joint>
     <xacro:unless value="${gazebo_visible}">
       <gazebo reference="${name}_cbf_volume">
@@ -99,8 +126,4 @@
       radius="0.075" length="0.24355" rgba="${arm_color}"
       gazebo_visible="${gazebo_visible}"/>
-    <xacro:cbf_sphere_visual
-      name="${prefix}elbow" parent="${prefix}forearm_link"
-      xyz="0 0 0" radius="0.075" rgba="${arm_color}"
-      gazebo_visible="${gazebo_visible}"/>
     <xacro:cbf_capsule_visual
       name="${prefix}forearm" parent="${prefix}forearm_link"
@@ -114,9 +137,7 @@
       Comprimento: 0.13105 - 0.027 = 0.10405 m.
     -->
-    <xacro:cbf_capsule_visual
+    <xacro:cbf_cylinder_visual
       name="${prefix}wrist_1_connector" parent="${prefix}forearm_link"
       center="-0.2132 0 0.079025" rpy="0 0 0"
-      cap_a="-0.2132 0 ${elbow_body_offset}"
-      cap_b="-0.2132 0 ${wrist_1_joint_offset}"
       radius="0.060" length="0.10405" rgba="${arm_color}"
       gazebo_visible="${gazebo_visible}"/>

Commit message: Fix Gazebo-only CBF volume visibility

File: ur_cbf_ws/src/ur_cbf_bringup/urdf/cbf_visual_volumes.urdf.xacro (robot description, xacro)
@@ -7,5 +7,5 @@
 <robot xmlns:xacro="http://wiki.ros.org/xacro">
   <xacro:macro name="cbf_sphere_visual"
-               params="name parent xyz radius rgba gazebo_visible">
+               params="name parent xyz radius rgba">
     <link name="${name}_cbf_volume">
       <visual name="${name}_cbf_visual">
@@ -24,16 +24,8 @@
       <child link="${name}_cbf_volume"/>
     </joint>
-    <!-- RViz ignora a extensao gazebo; visibility_flags=0 oculta somente no SDF. -->
-    <xacro:unless value="${gazebo_visible}">
-      <gazebo reference="${name}_cbf_volume">
-        <visual>
-          <visibility_flags>0</visibility_flags>
-        </visual>
-      </gazebo>
-    </xacro:unless>
   </xacro:macro>
   <!-- Cilindro sem tampas esfericas para ligar volumes ja sobrepostos. -->
   <xacro:macro name="cbf_cylinder_visual"
-               params="name parent center rpy radius length rgba gazebo_visible">
+               params="name parent center rpy radius length rgba">
     <link name="${name}_cbf_volume">
       <visual name="${name}_cbf_cylinder">
@@ -52,15 +44,8 @@
       <child link="${name}_cbf_volume"/>
     </joint>
-    <xacro:unless value="${gazebo_visible}">
-      <gazebo reference="${name}_cbf_volume">
-        <visual>
-          <visibility_flags>0</visibility_flags>
-        </visual>
-      </gazebo>
-    </xacro:unless>
   </xacro:macro>
   <!-- Uma capsula e formada por um cilindro e duas esferas, todos visuais. -->
   <xacro:macro name="cbf_capsule_visual"
-               params="name parent center rpy cap_a cap_b radius length rgba gazebo_visible">
+               params="name parent center rpy cap_a cap_b radius length rgba">
     <link name="${name}_cbf_volume">
       <visual name="${name}_cbf_cylinder">
@@ -93,13 +78,6 @@
       <child link="${name}_cbf_volume"/>
     </joint>
-    <xacro:unless value="${gazebo_visible}">
-      <gazebo reference="${name}_cbf_volume">
-        <visual>
-          <visibility_flags>0</visibility_flags>
-        </visual>
-      </gazebo>
-    </xacro:unless>
   </xacro:macro>
-  <xacro:macro name="ur3e_cbf_visual_volumes" params="prefix gazebo_visible">
+  <xacro:macro name="ur3e_cbf_visual_volumes" params="prefix">
     <xacro:property name="arm_color" value="0.00 0.75 1.00 0.25"/>
     <!--
@@ -113,10 +91,8 @@
     <xacro:cbf_sphere_visual
       name="${prefix}base" parent="${prefix}base_link"
-      xyz="0 0 0.075" radius="0.110" rgba="${arm_color}"
-      gazebo_visible="${gazebo_visible}"/>
+      xyz="0 0 0.075" radius="0.110" rgba="${arm_color}"/>
     <xacro:cbf_sphere_visual
       name="${prefix}shoulder" parent="${prefix}shoulder_link"
-      xyz="0 0 0" radius="0.090" rgba="${arm_color}"
-      gazebo_visible="${gazebo_visible}"/>
+      xyz="0 0 0" radius="0.090" rgba="${arm_color}"/>
     <xacro:cbf_capsule_visual
       name="${prefix}upper_arm" parent="${prefix}upper_arm_link"
@@ -124,6 +100,5 @@
       cap_a="0 0 ${shoulder_body_offset}"
       cap_b="-0.24355 0 ${shoulder_body_offset}"
-      radius="0.075" length="0.24355" rgba="${arm_color}"
-      gazebo_visible="${gazebo_visible}"/>
+      radius="0.075" length="0.24355" rgba="${arm_color}"/>
     <xacro:cbf_capsule_visual
       name="${prefix}forearm" parent="${prefix}forearm_link"
@@ -131,6 +106,5 @@
       cap_a="0 0 ${elbow_body_offset}"
       cap_b="-0.2132 0 ${elbow_body_offset}"
-      radius="0.065" length="0.2132" rgba="${arm_color}"
-      gazebo_visible="${gazebo_visible}"/>
+      radius="0.065" length="0.2132" rgba="${arm_color}"/>
     <!--
       Completa o offset distal do antebraco ate o frame posterior a junta 4.
@@ -140,20 +114,16 @@
       name="${prefix}wrist_1_connector" parent="${prefix}forearm_link"
       center="-0.2132 0 0.079025" rpy="0 0 0"
-      radius="0.060" length="0.10405" rgba="${arm_color}"
-      gazebo_visible="${gazebo_visible}"/>
+      radius="0.060" length="0.10405" rgba="${arm_color}"/>
     <xacro:cbf_sphere_visual
       name="${prefix}wrist_1" parent="${prefix}wrist_1_link"
-      xyz="0 0 0" radius="0.060" rgba="${arm_color}"
-      gazebo_visible="${gazebo_visible}"/>
+      xyz="0 0 0" radius="0.060" rgba="${arm_color}"/>
     <xacro:cbf_sphere_visual
       name="${prefix}wrist_2" parent="${prefix}wrist_2_link"
-      xyz="0 0 0" radius="0.058" rgba="${arm_color}"
-      gazebo_visible="${gazebo_visible}"/>
+      xyz="0 0 0" radius="0.058" rgba="${arm_color}"/>
     <xacro:cbf_sphere_visual
       name="${prefix}wrist_3" parent="${prefix}wrist_3_link"
-      xyz="0 0 0" radius="0.058" rgba="${arm_color}"
-      gazebo_visible="${gazebo_visible}"/>
+      xyz="0 0 0" radius="0.058" rgba="${arm_color}"/>
   </xacro:macro>
-  <xacro:macro name="rg2_cbf_visual_volume" params="prefix gazebo_visible">
+  <xacro:macro name="rg2_cbf_visual_volume" params="prefix">
     <!-- Uma unica capsula cobre corpo, dedos e o TCP nominal da RG2. -->
     <xacro:cbf_capsule_visual
@@ -161,6 +131,5 @@
       center="0 0 0.110" rpy="0 0 0"
       cap_a="0 0 0.055" cap_b="0 0 0.165"
-      radius="0.090" length="0.110" rgba="1.00 0.45 0.00 0.30"
-      gazebo_visible="${gazebo_visible}"/>
+      radius="0.090" length="0.110" rgba="1.00 0.45 0.00 0.30"/>
   </xacro:macro>
 </robot>

File: ur_cbf_ws/src/ur_cbf_bringup/urdf/ur_rg2_gz.urdf.xacro (robot description, xacro)
@@ -20,5 +20,4 @@
   <xacro:arg name="ros_namespace" default=""/>
   <xacro:arg name="show_cbf_volumes" default="$(optenv CBF_VOLUMES true)"/>
-  <xacro:arg name="show_cbf_volumes_gazebo" default="$(optenv CBF_VOLUMES_GAZEBO true)"/>
   <!-- O Xacro upstream declara gripper_tcp no escopo da inclusao. -->
   <xacro:property name="prefix" value="$(arg tf_prefix)"/>
@@ -64,10 +63,8 @@
     <xacro:if value="${selected_ur_type == 'ur3e'}">
       <xacro:ur3e_cbf_visual_volumes
-        prefix="$(arg tf_prefix)"
-        gazebo_visible="$(arg show_cbf_volumes_gazebo)"/>
+        prefix="$(arg tf_prefix)"/>
     </xacro:if>
     <xacro:rg2_cbf_visual_volume
-      prefix="$(arg tf_prefix)"
-      gazebo_visible="$(arg show_cbf_volumes_gazebo)"/>
+      prefix="$(arg tf_prefix)"/>
   </xacro:if>
   <gazebo reference="world"/>

File: ur_cbf_ws/src/ur_cbf_bringup/urdf/ur_rg6_gz.urdf.xacro (robot description, xacro)
@@ -20,5 +20,4 @@
   <xacro:arg name="ros_namespace" default=""/>
   <xacro:arg name="show_cbf_volumes" default="$(optenv CBF_VOLUMES true)"/>
-  <xacro:arg name="show_cbf_volumes_gazebo" default="$(optenv CBF_VOLUMES_GAZEBO true)"/>
   <!-- O Xacro upstream declara gripper_tcp no escopo da inclusao. -->
   <xacro:property name="prefix" value="$(arg tf_prefix)"/>
@@ -64,6 +63,5 @@
     <xacro:if value="${selected_ur_type == 'ur3e'}">
       <xacro:ur3e_cbf_visual_volumes
-        prefix="$(arg tf_prefix)"
-        gazebo_visible="$(arg show_cbf_volumes_gazebo)"/>
+        prefix="$(arg tf_prefix)"/>
     </xacro:if>
   </xacro:if>
