Commit message: Add UAIbot self-collision CBF geometry

File: ur_cbf_ws/src/ur_cbf_bringup/urdf/cbf_visual_volumes.urdf.xacro (robot description, xacro)
@@ -1,5 +1,12 @@
 <?xml version="1.0"?>
 <!--
-  Aproximacoes geometricas visuais para inspecao das futuras CBFs.
+  Copia visual dos objetos de colisao internos do UAIbot 1.2.7 para o UR3e.
+  Fonte fixada:
+  UAIbot/UAIbotPy@1acb5ed637738aca4ea05945e6c065c3757bc13d
+  uaibot/robot/_create_ur_ur3e.py
+  As matrizes htm_obj do UAIbot sao relativas aos frames DH posteriores a cada
+  junta. Os origins abaixo aplicam as transformacoes rigidas DH -> elo URDF da
+  descricao oficial Jazzy. Cilindros usam o eixo local z; caixas usam
+  width/depth/height como x/y/z, igualmente ao UAIbot.
   Estes links nao possuem collision nem inertial: aparecem no RViz e no Gazebo,
   acompanham os elos por juntas fixas e nao alteram a fisica da simulacao.
@@ -25,10 +32,9 @@
     </joint>
   </xacro:macro>
-  <!-- Cilindro sem tampas esfericas para ligar volumes ja sobrepostos. -->
   <xacro:macro name="cbf_cylinder_visual"
-               params="name parent center rpy radius length rgba">
+               params="name parent xyz rpy radius length rgba">
     <link name="${name}_cbf_volume">
-      <visual name="${name}_cbf_cylinder">
-        <origin xyz="${center}" rpy="${rpy}"/>
+      <visual name="${name}_cbf_visual">
+        <origin xyz="${xyz}" rpy="${rpy}"/>
         <geometry>
           <cylinder radius="${radius}" length="${length}"/>
@@ -45,30 +51,15 @@
     </joint>
   </xacro:macro>
-  <!-- Uma capsula e formada por um cilindro e duas esferas, todos visuais. -->
-  <xacro:macro name="cbf_capsule_visual"
-               params="name parent center rpy cap_a cap_b radius length rgba">
+  <xacro:macro name="cbf_box_visual"
+               params="name parent xyz rpy size rgba">
     <link name="${name}_cbf_volume">
-      <visual name="${name}_cbf_cylinder">
-        <origin xyz="${center}" rpy="${rpy}"/>
+      <visual name="${name}_cbf_visual">
+        <origin xyz="${xyz}" rpy="${rpy}"/>
         <geometry>
-          <cylinder radius="${radius}" length="${length}"/>
+          <box size="${size}"/>
         </geometry>
         <material name="${name}_cbf_material">
           <color rgba="${rgba}"/>
         </material>
-      </visual>
-      <visual name="${name}_cbf_cap_a">
-        <origin xyz="${cap_a}" rpy="0 0 0"/>
-        <geometry>
-          <sphere radius="${radius}"/>
-        </geometry>
-        <material name="${name}_cbf_material"/>
-      </visual>
-      <visual name="${name}_cbf_cap_b">
-        <origin xyz="${cap_b}" rpy="0 0 0"/>
-        <geometry>
-          <sphere radius="${radius}"/>
-        </geometry>
-        <material name="${name}_cbf_material"/>
       </visual>
     </link>
@@ -81,55 +72,85 @@
   <xacro:macro name="ur3e_cbf_visual_volumes" params="prefix">
     <xacro:property name="arm_color" value="0.00 0.75 1.00 0.25"/>
-    <!--
-      Offsets fisicos da descricao oficial Jazzy do UR3e. Os eixos DH passam
-      pelas juntas, enquanto os corpos do braco e antebraco sao deslocados em z
-      nos respectivos frames de elo.
-    -->
-    <xacro:property name="shoulder_body_offset" value="0.120"/>
-    <xacro:property name="elbow_body_offset" value="0.027"/>
-    <xacro:property name="wrist_1_joint_offset" value="0.13105"/>
+    <xacro:property name="tool_color" value="1.00 0.45 0.00 0.30"/>
+    <!-- UAIbot link 0; ^shoulder_link T_DH0 = Rx(pi/2). -->
+    <xacro:cbf_cylinder_visual
+      name="${prefix}uaibot_c0" parent="${prefix}shoulder_link"
+      xyz="0 0 -0.0469" rpy="0 0 0"
+      radius="0.067" length="0.21" rgba="${arm_color}"/>
+    <!-- UAIbot link 1; ^upper_arm_link T_DH1 = Tx(-0.24355). -->
+    <xacro:cbf_cylinder_visual
+      name="${prefix}uaibot_c11" parent="${prefix}upper_arm_link"
+      xyz="0.00185 0 0.118" rpy="0 0 1.570796326795"
+      radius="0.052" length="0.13" rgba="${arm_color}"/>
+    <xacro:cbf_cylinder_visual
+      name="${prefix}uaibot_c12" parent="${prefix}upper_arm_link"
+      xyz="-0.11815 0 0.12" rpy="-1.570796326795 0 1.570796326795"
+      radius="0.05" length="0.2" rgba="${arm_color}"/>
+    <xacro:cbf_cylinder_visual
+      name="${prefix}uaibot_c13" parent="${prefix}upper_arm_link"
+      xyz="-0.24315 0 0.118" rpy="0 0 1.570796326795"
+      radius="0.05" length="0.12" rgba="${arm_color}"/>
+    <!-- UAIbot link 2; ^forearm_link T_DH2 = Tx(-0.2132). -->
     <xacro:cbf_sphere_visual
-      name="${prefix}base" parent="${prefix}base_link"
-      xyz="0 0 0.075" radius="0.110" rgba="${arm_color}"/>
+      name="${prefix}uaibot_c21" parent="${prefix}forearm_link"
+      xyz="-0.0246 0 0.05" radius="0.05" rgba="${arm_color}"/>
+    <xacro:cbf_cylinder_visual
+      name="${prefix}uaibot_c22" parent="${prefix}forearm_link"
+      xyz="-0.1046 0 0.05" rpy="-1.570796326795 0 1.570796326795"
+      radius="0.04" length="0.2" rgba="${arm_color}"/>
+    <xacro:cbf_cylinder_visual
+      name="${prefix}uaibot_c23" parent="${prefix}forearm_link"
+      xyz="-0.2146 0 0.045" rpy="0 0 1.570796326795"
+      radius="0.035" length="0.09" rgba="${arm_color}"/>
+    <!-- UAIbot link 3; ^wrist_1_link T_DH3 = Rx(pi/2). -->
+    <xacro:cbf_cylinder_visual
+      name="${prefix}uaibot_c31" parent="${prefix}wrist_1_link"
+      xyz="0 -0.0014 0.0039" rpy="0 0 3.14159265359"
+      radius="0.035" length="0.09" rgba="${arm_color}"/>
+    <xacro:cbf_cylinder_visual
+      name="${prefix}uaibot_c32" parent="${prefix}wrist_1_link"
+      xyz="0 -0.0414 -0.0011" rpy="-1.570796326795 0 -3.14159265359"
+      radius="0.035" length="0.045" rgba="${arm_color}"/>
+    <!-- UAIbot link 4; ^wrist_2_link T_DH4 = Rx(-pi/2). -->
+    <xacro:cbf_cylinder_visual
+      name="${prefix}uaibot_c41" parent="${prefix}wrist_2_link"
+      xyz="0.0011 0 -0.034" rpy="0 0 -1.570796326795"
+      radius="0.035" length="0.025" rgba="${arm_color}"/>
+    <xacro:cbf_cylinder_visual
+      name="${prefix}uaibot_c42" parent="${prefix}wrist_2_link"
+      xyz="0.0011 -0.0025 -0.004" rpy="1.570796326795 1.570796326795 0"
+      radius="0.038" length="0.098" rgba="${arm_color}"/>
+    <!-- UAIbot link 5; ^wrist_3_link T_DH5 = I. -->
+    <xacro:cbf_cylinder_visual
+      name="${prefix}uaibot_c51" parent="${prefix}wrist_3_link"
+      xyz="0.0011 0.004 -0.0231" rpy="3.14159265359 0 1.570796326795"
+      radius="0.038" length="0.046" rgba="${arm_color}"/>
+    <xacro:cbf_cylinder_visual
+      name="${prefix}uaibot_c52" parent="${prefix}wrist_3_link"
+      xyz="0.0011 -0.021 -0.0201" rpy="1.570796326795 1.570796326795 0"
+      radius="0.01" length="0.028" rgba="${arm_color}"/>
     <xacro:cbf_sphere_visual
-      name="${prefix}shoulder" parent="${prefix}shoulder_link"
-      xyz="0 0 0" radius="0.090" rgba="${arm_color}"/>
-    <xacro:cbf_capsule_visual
-      name="${prefix}upper_arm" parent="${prefix}upper_arm_link"
-      center="-0.121775 0 ${shoulder_body_offset}" rpy="0 1.57079632679 0"
-      cap_a="0 0 ${shoulder_body_offset}"
-      cap_b="-0.24355 0 ${shoulder_body_offset}"
-      radius="0.075" length="0.24355" rgba="${arm_color}"/>
-    <xacro:cbf_capsule_visual
-      name="${prefix}forearm" parent="${prefix}forearm_link"
-      center="-0.1066 0 ${elbow_body_offset}" rpy="0 1.57079632679 0"
-      cap_a="0 0 ${elbow_body_offset}"
-      cap_b="-0.2132 0 ${elbow_body_offset}"
-      radius="0.065" length="0.2132" rgba="${arm_color}"/>
-    <!--
-      Completa o offset distal do antebraco ate o frame posterior a junta 4.
-      Comprimento: 0.13105 - 0.027 = 0.10405 m.
-    -->
+      name="${prefix}uaibot_c53" parent="${prefix}wrist_3_link"
+      xyz="0.0011 0.004 0.0279" radius="0.05" rgba="${tool_color}"/>
+    <xacro:cbf_box_visual
+      name="${prefix}uaibot_c54" parent="${prefix}wrist_3_link"
+      xyz="0.0011 -0.006 0.1079" rpy="1.570796326795 1.570796326795 0"
+      size="0.09 0.07 0.06" rgba="${tool_color}"/>
+    <xacro:cbf_box_visual
+      name="${prefix}uaibot_c55" parent="${prefix}wrist_3_link"
+      xyz="-0.0389 -0.001 0.1529" rpy="1.570796326795 0.785398163397 0"
+      size="0.075 0.04 0.035" rgba="${tool_color}"/>
+    <xacro:cbf_box_visual
+      name="${prefix}uaibot_c56" parent="${prefix}wrist_3_link"
+      xyz="0.0411 -0.001 0.1529" rpy="-1.570796326795 0.785398163397 -3.14159265359"
+      size="0.075 0.04 0.035" rgba="${tool_color}"/>
     <xacro:cbf_cylinder_visual
-      name="${prefix}wrist_1_connector" parent="${prefix}forearm_link"
-      center="-0.2132 0 0.079025" rpy="0 0 0"
-      radius="0.060" length="0.10405" rgba="${arm_color}"/>
-    <xacro:cbf_sphere_visual
-      name="${prefix}wrist_1" parent="${prefix}wrist_1_link"
-      xyz="0 0 0" radius="0.060" rgba="${arm_color}"/>
-    <xacro:cbf_sphere_visual
-      name="${prefix}wrist_2" parent="${prefix}wrist_2_link"
-      xyz="0 0 0" radius="0.058" rgba="${arm_color}"/>
-    <xacro:cbf_sphere_visual
-      name="${prefix}wrist_3" parent="${prefix}wrist_3_link"
-      xyz="0 0 0" radius="0.058" rgba="${arm_color}"/>
-  </xacro:macro>
-  <xacro:macro name="rg2_cbf_visual_volume" params="prefix">
-    <!-- Uma unica capsula cobre corpo, dedos e o TCP nominal da RG2. -->
-    <xacro:cbf_capsule_visual
-      name="${prefix}rg2" parent="${prefix}onrobot_base_link"
-      center="0 0 0.110" rpy="0 0 0"
-      cap_a="0 0 0.055" cap_b="0 0 0.165"
-      radius="0.090" length="0.110" rgba="1.00 0.45 0.00 0.30"/>
+      name="${prefix}uaibot_c57" parent="${prefix}wrist_3_link"
+      xyz="0.0511 -0.001 0.1979" rpy="3.14159265359 0 1.570796326795"
+      radius="0.021" length="0.04" rgba="${tool_color}"/>
+    <xacro:cbf_cylinder_visual
+      name="${prefix}uaibot_c58" parent="${prefix}wrist_3_link"
+      xyz="-0.0489 -0.001 0.1979" rpy="3.14159265359 0 1.570796326795"
+      radius="0.021" length="0.04" rgba="${tool_color}"/>
   </xacro:macro>
 </robot>

File: ur_cbf_ws/src/ur_cbf_bringup/urdf/ur_rg2_gz.urdf.xacro (robot description, xacro)
@@ -65,6 +65,4 @@
         prefix="$(arg tf_prefix)"/>
     </xacro:if>
-    <xacro:rg2_cbf_visual_volume
-      prefix="$(arg tf_prefix)"/>
   </xacro:if>
   <gazebo reference="world"/>

Commit message: Apply corrected UR3e RG2 collision geometry

File: ur_cbf_ws/src/ur_cbf_bringup/urdf/cbf_visual_volumes.urdf.xacro (robot description, xacro)
@@ -1,12 +1,13 @@
 <?xml version="1.0"?>
 <!--
-  Copia visual dos objetos de colisao internos do UAIbot 1.2.7 para o UR3e.
+  Modelo visual de autocolisao corrigido do projeto para o conjunto UR3e/RG2.
   Fonte fixada:
   UAIbot/UAIbotPy@1acb5ed637738aca4ea05945e6c065c3757bc13d
   uaibot/robot/_create_ur_ur3e.py
-  As matrizes htm_obj do UAIbot sao relativas aos frames DH posteriores a cada
-  junta. Os origins abaixo aplicam as transformacoes rigidas DH -> elo URDF da
-  descricao oficial Jazzy. Cilindros usam o eixo local z; caixas usam
-  width/depth/height como x/y/z, igualmente ao UAIbot.
+  Os treze objetos do UR3e preservados da fabrica UAIbot sao relativos aos
+  frames DH posteriores a cada junta. Os origins abaixo aplicam as
+  transformacoes rigidas DH -> elo URDF da descricao oficial Jazzy. A garra
+  generica da dependencia foi substituida por uma capsula RG2 pertencente ao
+  projeto, formada por um cilindro e duas esferas.
   Estes links nao possuem collision nem inertial: aparecem no RViz e no Gazebo,
   acompanham os elos por juntas fixas e nao alteram a fisica da simulacao.
@@ -51,15 +52,29 @@
     </joint>
   </xacro:macro>
-  <xacro:macro name="cbf_box_visual"
-               params="name parent xyz rpy size rgba">
+  <xacro:macro name="cbf_capsule_visual"
+               params="name parent center rpy cap_a cap_b radius length rgba">
     <link name="${name}_cbf_volume">
-      <visual name="${name}_cbf_visual">
-        <origin xyz="${xyz}" rpy="${rpy}"/>
+      <visual name="${name}_cbf_cylinder">
+        <origin xyz="${center}" rpy="${rpy}"/>
         <geometry>
-          <box size="${size}"/>
+          <cylinder radius="${radius}" length="${length}"/>
         </geometry>
         <material name="${name}_cbf_material">
           <color rgba="${rgba}"/>
         </material>
+      </visual>
+      <visual name="${name}_cbf_cap_a">
+        <origin xyz="${cap_a}" rpy="0 0 0"/>
+        <geometry>
+          <sphere radius="${radius}"/>
+        </geometry>
+        <material name="${name}_cbf_material"/>
+      </visual>
+      <visual name="${name}_cbf_cap_b">
+        <origin xyz="${cap_b}" rpy="0 0 0"/>
+        <geometry>
+          <sphere radius="${radius}"/>
+        </geometry>
+        <material name="${name}_cbf_material"/>
       </visual>
     </link>
@@ -72,5 +87,4 @@
   <xacro:macro name="ur3e_cbf_visual_volumes" params="prefix">
     <xacro:property name="arm_color" value="0.00 0.75 1.00 0.25"/>
-    <xacro:property name="tool_color" value="1.00 0.45 0.00 0.30"/>
     <!-- UAIbot link 0; ^shoulder_link T_DH0 = Rx(pi/2). -->
     <xacro:cbf_cylinder_visual
@@ -130,27 +144,12 @@
       xyz="0.0011 -0.021 -0.0201" rpy="1.570796326795 1.570796326795 0"
       radius="0.01" length="0.028" rgba="${arm_color}"/>
-    <xacro:cbf_sphere_visual
-      name="${prefix}uaibot_c53" parent="${prefix}wrist_3_link"
-      xyz="0.0011 0.004 0.0279" radius="0.05" rgba="${tool_color}"/>
-    <xacro:cbf_box_visual
-      name="${prefix}uaibot_c54" parent="${prefix}wrist_3_link"
-      xyz="0.0011 -0.006 0.1079" rpy="1.570796326795 1.570796326795 0"
-      size="0.09 0.07 0.06" rgba="${tool_color}"/>
-    <xacro:cbf_box_visual
-      name="${prefix}uaibot_c55" parent="${prefix}wrist_3_link"
-      xyz="-0.0389 -0.001 0.1529" rpy="1.570796326795 0.785398163397 0"
-      size="0.075 0.04 0.035" rgba="${tool_color}"/>
-    <xacro:cbf_box_visual
-      name="${prefix}uaibot_c56" parent="${prefix}wrist_3_link"
-      xyz="0.0411 -0.001 0.1529" rpy="-1.570796326795 0.785398163397 -3.14159265359"
-      size="0.075 0.04 0.035" rgba="${tool_color}"/>
-    <xacro:cbf_cylinder_visual
-      name="${prefix}uaibot_c57" parent="${prefix}wrist_3_link"
-      xyz="0.0511 -0.001 0.1979" rpy="3.14159265359 0 1.570796326795"
-      radius="0.021" length="0.04" rgba="${tool_color}"/>
-    <xacro:cbf_cylinder_visual
-      name="${prefix}uaibot_c58" parent="${prefix}wrist_3_link"
-      xyz="-0.0489 -0.001 0.1979" rpy="3.14159265359 0 1.570796326795"
-      radius="0.021" length="0.04" rgba="${tool_color}"/>
+  </xacro:macro>
+  <xacro:macro name="rg2_cbf_visual_volume" params="prefix">
+    <!-- Mesmos tres objetos anexados ao ultimo elo do modelo UAIbot corrigido. -->
+    <xacro:cbf_capsule_visual
+      name="${prefix}rg2" parent="${prefix}onrobot_base_link"
+      center="0 0 0.110" rpy="0 0 0"
+      cap_a="0 0 0.055" cap_b="0 0 0.165"
+      radius="0.090" length="0.110" rgba="1.00 0.45 0.00 0.30"/>
   </xacro:macro>
 </robot>

File: ur_cbf_ws/src/ur_cbf_bringup/urdf/ur_rg2_gz.urdf.xacro (robot description, xacro)
@@ -64,4 +64,5 @@
       <xacro:ur3e_cbf_visual_volumes
         prefix="$(arg tf_prefix)"/>
+      <xacro:rg2_cbf_visual_volume prefix="$(arg tf_prefix)"/>
     </xacro:if>
   </xacro:if>

Commit message: Simplifica garra RG2 para dois volumes

File: ur_cbf_ws/src/ur_cbf_bringup/urdf/cbf_visual_volumes.urdf.xacro (robot description, xacro)
@@ -13,5 +13,5 @@
   y=0 m e comprimento=0.0945 m; c41 usa z=-0.027 m; c42 usa
   x=0, y=0 m e z=0; c51 permanece inalterado; e c52 usa x=0.0011 m, y=-0.026 m e z=-0.030 m.
-  A garra generica foi substituida por uma capsula RG2 pertencente ao projeto.
+  A garra generica foi substituida por dois volumes RG2 pertencentes ao projeto.
   Estes links nao possuem collision nem inertial: aparecem no RViz e no Gazebo,
   acompanham os elos por juntas fixas e nao alteram a fisica da simulacao.
@@ -56,11 +56,11 @@
     </joint>
   </xacro:macro>
-  <xacro:macro name="cbf_capsule_visual"
-               params="name parent center rpy cap_a cap_b radius length rgba">
+  <xacro:macro name="cbf_cylinder_sphere_visual"
+               params="name parent center rpy sphere_center cylinder_radius sphere_radius length rgba">
     <link name="${name}_cbf_volume">
       <visual name="${name}_cbf_cylinder">
         <origin xyz="${center}" rpy="${rpy}"/>
         <geometry>
-          <cylinder radius="${radius}" length="${length}"/>
+          <cylinder radius="${cylinder_radius}" length="${length}"/>
         </geometry>
         <material name="${name}_cbf_material">
@@ -68,15 +68,8 @@
         </material>
       </visual>
-      <visual name="${name}_cbf_cap_a">
-        <origin xyz="${cap_a}" rpy="0 0 0"/>
+      <visual name="${name}_cbf_sphere">
+        <origin xyz="${sphere_center}" rpy="0 0 0"/>
         <geometry>
-          <sphere radius="${radius}"/>
-        </geometry>
-        <material name="${name}_cbf_material"/>
-      </visual>
-      <visual name="${name}_cbf_cap_b">
-        <origin xyz="${cap_b}" rpy="0 0 0"/>
-        <geometry>
-          <sphere radius="${radius}"/>
+          <sphere radius="${sphere_radius}"/>
         </geometry>
         <material name="${name}_cbf_material"/>
@@ -150,10 +143,11 @@
   </xacro:macro>
   <xacro:macro name="rg2_cbf_visual_volume" params="prefix">
-    <!-- Mesmos tres objetos anexados ao ultimo elo do modelo UAIbot corrigido. -->
-    <xacro:cbf_capsule_visual
+    <!-- Dois objetos: cilindro com o diametro de C51 e esfera terminal. -->
+    <xacro:cbf_cylinder_sphere_visual
       name="${prefix}rg2" parent="${prefix}onrobot_base_link"
       center="0 0 0.110" rpy="0 0 0"
-      cap_a="0 0 0.055" cap_b="0 0 0.165"
-      radius="0.090" length="0.110" rgba="1.00 0.45 0.00 0.30"/>
+      sphere_center="0 0 0.165"
+      cylinder_radius="0.038" sphere_radius="0.090"
+      length="0.110" rgba="1.00 0.45 0.00 0.30"/>
   </xacro:macro>
 </robot>

Commit message: Simplifica manipulacao e restaura volumes RG2 do UAIbot

File: ur_cbf_ws/src/ur_cbf_bringup/urdf/cbf_visual_volumes.urdf.xacro (robot description, xacro)
@@ -13,5 +13,7 @@
   y=0 m e comprimento=0.0945 m; c41 usa z=-0.027 m; c42 usa
   x=0, y=0 m e z=0; c51 permanece inalterado; e c52 usa x=0.0011 m, y=-0.026 m e z=-0.030 m.
-  A garra generica foi substituida por dois volumes RG2 pertencentes ao projeto.
+  A RG2 usa os oito objetos do elo final da fabrica UAIbot: C51/C52 e os seis
+  objetos adicionais de esfera, caixas e cilindros. Estes links sao apenas
+  visuais e permanecem sincronizados com UR3E_RG2_PROJECT_PRIMITIVES.
   Estes links nao possuem collision nem inertial: aparecem apenas na descricao
   visual usada pelo RViz, acompanham os elos por juntas fixas e nao alteram a
@@ -57,22 +59,15 @@
     </joint>
   </xacro:macro>
-  <xacro:macro name="cbf_cylinder_sphere_visual"
-               params="name parent center rpy sphere_center cylinder_radius sphere_radius length rgba">
+  <xacro:macro name="cbf_box_visual"
+               params="name parent xyz rpy size rgba">
     <link name="${name}_cbf_volume">
-      <visual name="${name}_cbf_cylinder">
-        <origin xyz="${center}" rpy="${rpy}"/>
+      <visual name="${name}_cbf_visual">
+        <origin xyz="${xyz}" rpy="${rpy}"/>
         <geometry>
-          <cylinder radius="${cylinder_radius}" length="${length}"/>
+          <box size="${size}"/>
         </geometry>
         <material name="${name}_cbf_material">
           <color rgba="${rgba}"/>
         </material>
-      </visual>
-      <visual name="${name}_cbf_sphere">
-        <origin xyz="${sphere_center}" rpy="0 0 0"/>
-        <geometry>
-          <sphere radius="${sphere_radius}"/>
-        </geometry>
-        <material name="${name}_cbf_material"/>
       </visual>
     </link>
@@ -144,11 +139,31 @@
   </xacro:macro>
   <xacro:macro name="rg2_cbf_visual_volume" params="prefix">
-    <!-- Dois objetos: cilindro com o diametro de C51 e esfera terminal. -->
-    <xacro:cbf_cylinder_sphere_visual
-      name="${prefix}rg2" parent="${prefix}onrobot_base_link"
-      center="0 0 0.050" rpy="0 0 0"
-      sphere_center="0 0 0.165"
-      cylinder_radius="0.048" sphere_radius="0.090"
-      length="0.110" rgba="1.00 0.45 0.00 0.30"/>
+    <!-- Objetos 2..7 do elo 5 original do UAIbot, no frame wrist_3_link. -->
+    <xacro:cbf_sphere_visual
+      name="${prefix}uaibot_c53" parent="${prefix}wrist_3_link"
+      xyz="0.0011 0.004 0.0279" radius="0.05"
+      rgba="1.00 0.45 0.00 0.30"/>
+    <xacro:cbf_box_visual
+      name="${prefix}uaibot_c54" parent="${prefix}wrist_3_link"
+      xyz="0.0011 -0.006 0.1079" rpy="0 1.570796326795 0"
+      size="0.09 0.07 0.06" rgba="1.00 0.45 0.00 0.30"/>
+    <xacro:cbf_box_visual
+      name="${prefix}uaibot_c55" parent="${prefix}wrist_3_link"
+      xyz="-0.0389 -0.001 0.1529"
+      rpy="1.570796326795 0.785398163397 0"
+      size="0.075 0.04 0.035" rgba="1.00 0.45 0.00 0.30"/>
+    <xacro:cbf_box_visual
+      name="${prefix}uaibot_c56" parent="${prefix}wrist_3_link"
+      xyz="0.0411 -0.001 0.1529"
+      rpy="-1.570796326795 0.785398163397 3.14159265359"
+      size="0.075 0.04 0.035" rgba="1.00 0.45 0.00 0.30"/>
+    <xacro:cbf_cylinder_visual
+      name="${prefix}uaibot_c57" parent="${prefix}wrist_3_link"
+      xyz="0.0511 -0.001 0.1979" rpy="3.14159265359 0 1.570796326795"
+      radius="0.021" length="0.04" rgba="1.00 0.45 0.00 0.30"/>
+    <xacro:cbf_cylinder_visual
+      name="${prefix}uaibot_c58" parent="${prefix}wrist_3_link"
+      xyz="-0.0489 -0.001 0.1979" rpy="3.14159265359 0 1.570796326795"
+      radius="0.021" length="0.04" rgba="1.00 0.45 0.00 0.30"/>
   </xacro:macro>
 </robot>
