Commit message: Corrige modelos estaticos e adiciona piso da cena

File: ur_cbf_ws/src/ur_cbf_bringup/worlds/manipulation.sdf.xacro (robot description, xacro)
@@ -39,5 +39,31 @@
       <specular>0.2 0.2 0.2 1</specular>
     </light>
-    <model name="manipulation_table" static="true">
+    <model name="ground_plane">
+      <static>true</static>
+      <link name="ground_link">
+        <collision name="ground_collision">
+          <geometry>
+            <plane>
+              <normal>0 0 1</normal>
+              <size>10 10</size>
+            </plane>
+          </geometry>
+        </collision>
+        <visual name="ground_visual">
+          <geometry>
+            <plane>
+              <normal>0 0 1</normal>
+              <size>10 10</size>
+            </plane>
+          </geometry>
+          <material>
+            <ambient>0.18 0.18 0.18 1</ambient>
+            <diffuse>0.25 0.25 0.25 1</diffuse>
+          </material>
+        </visual>
+      </link>
+    </model>
+    <model name="manipulation_table">
+      <static>true</static>
       <pose>$(arg table_x) $(arg table_y) $(arg table_z) 0 0 0</pose>
       <link name="table_link">
@@ -93,5 +119,6 @@
       </link>
     </model>
-    <model name="drop_box" static="true">
+    <model name="drop_box">
+      <static>true</static>
       <pose>$(arg drop_x) $(arg drop_y) 0 0 0 0</pose>
       <link name="box_link">
